File: Satellite Platform PCB/Project_PCB.brd (EAGLE design)
At the start: 115.5 x 68.2 mm, 32 parts, among them IC1 A4990KLPTR-T, IC4 A4990KLPTR-T

Commit message: approved DRC errors
Routing:
- net GND: track 50.9 -> 43.9 mm
Changed lines of the file:
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@@
 <wire x1="33.02" y1="13.259" x2="39.929" y2="13.259" width="0.8128" layer="1"/>
 <wire x1="39.929" y1="13.259" x2="41.91" y2="15.24" width="0.8128" layer="1"/>
-<wire x1="14.859" y1="22.098" x2="14.859" y2="29.1372" width="0.4064" layer="16"/>
 <wire x1="14.859" y1="29.1372" x2="15.113" y2="29.3912" width="0.4064" layer="16"/>
 <via x="15.113" y="29.3912" extent="1-16" drill="0.35"/>
@@
 <mfgpreviewcolor name="substratecolor" color="0xFF786E46"/>
 </mfgpreviewcolors>
+<errors>
+</errors>
 </board>
 </drawing>

Commit message: gerber folder made
Routing:
- net GND: track 43.9 -> 33.8 mm, vias 11 -> 43
- net N$42: track 30.1 -> 24.7 mm
- net N$43: track 30.7 -> 26.8 mm
- net N$46: track 76.0 -> 72.9 mm, vias 2 -> 6
- added copper zone on layer 1, net GND
- removed copper zone on layer 1, net HEAT_1
- removed copper zone on layer 16, net HEAT_1
- removed copper zone on layer 1, net HEAT_2
- removed copper zone on layer 16, net HEAT_2

Commit message: pcb gerber
Routing:
- net N$8: track 45.6 -> 44.8 mm
- net N$7: track 36.4 -> 35.7 mm
- net N$21: track 110.3 -> 109.6 mm
